Commit message: Add realsense_gazebo_sim

File: robot_sim_gazebo/sensor/navigation_platform.xacro (robot description, xacro)
@@ -11,4 +11,6 @@
     <xacro:arg name="imu" default="false" />
     <xacro:arg name="gps" default="false" />
+    <xacro:arg name="d435" default="false" />
+    <xacro:arg name="t265" default="false" />
     <xacro:property name="gpu" value="$(arg gpu)" />
     <xacro:property name="lidar" value="$(arg lidar)" />
@@ -16,4 +18,6 @@
     <xacro:property name="imu" value="$(arg imu)" />
     <xacro:property name="gps" value="$(arg gps)" />
+    <xacro:property name="d435" value="$(arg d435)" />
+    <xacro:property name="t265" value="$(arg t265)" />
     <xacro:if value="${lidar}">
         <xacro:include filename="$(find robot_sim_gazebo)/sensor/lidar_robot.urdf.xacro"
@@ -29,3 +33,9 @@
         <xacro:include filename="$(find robot_sim_gazebo)/sensor/gps.xacro" />
     </xacro:if>
+    <xacro:if value="${d435}">
+        <xacro:include filename="$(find robot_sim_gazebo)/sensor/realsense_d435.xacro" />
+    </xacro:if>
+    <xacro:if value="${t265}">
+        <xacro:include filename="$(find robot_sim_gazebo)/sensor/realsense_t265.xacro" />
+    </xacro:if>
 </robot>
